File: CarrierBoard/PiProjector.brd (EAGLE design)
At the start: 86.4 x 54.6 mm, 73 parts, among them P8 PINHEAD2X23, P9 PINHEAD2X23, X1 24MHz, X2 12Mhz

Commit message: POE connection Moved
Started Modification for Adjusted POE connection
Parts:
- removed AUX_BTN: (no value), pinhead:2X04
Connections:
- removed net MUTEP: AUX_BTN.4, U$6.18
- removed net MUTEREC: AUX_BTN.8, U$6.6
- removed net VOLDN: AUX_BTN.6, U$6.48
- removed net VOLUP: AUX_BTN.2, U$6.39
- new net MUTP: P8.7, U$6.18
- new net MUTR: P8.8, U$6.6
- new net VLDN: P8.10, U$6.48
- new net VLUP: P8.9, U$6.39
- net +5V: now also P8.3, P8.4; no longer AUX_BTN.5
- net GND: now also P8.1, P8.2; no longer AUX_BTN.7
- net POE+: now also P8.5; no longer AUX_BTN.1
- net POE-: now also P8.6; no longer AUX_BTN.3
Routing:
- net VOLUP: track 17.5 -> 0.00 mm
- net VOLDN: track 17.5 -> 0.00 mm
- net POE-: track 24.8 -> 40.8 mm
- net MUTEREC: track 15.8 -> 0.00 mm
- net POE+: track 19.5 -> 34.2 mm
- net MUTEP: track 8.60 -> 0.00 mm
- net +5V: track 68.8 -> 66.7 mm

Commit message: Finished modified daughterboard
Routing:
- net MUTR: track 0.00 -> 52.4 mm, vias 0 -> 1
- net VLDN: track 0.00 -> 51.1 mm, vias 0 -> 1
- net VLUP: track 0.00 -> 43.8 mm, vias 0 -> 1
- net MUTP: track 0.00 -> 40.5 mm, vias 0 -> 3
- net USB5D_P: track 90.4 -> 94.5 mm
- net USB5D_N: track 89.8 -> 93.9 mm

Commit message: minor fix
Parts:
- moved C9 2.31 mm to (-32.7, -10.5)
- moved C15 0.10 mm to (-16.5, -17.9)
- moved C14 0.10 mm to (-11.9, -17.9)
Routing:
- net GND: track 231.0 -> 232.5 mm, vias 60 -> 59
- net VBUS: track 147.6 -> 148.4 mm
Other:
- board text removed: "+5V"
- board text removed: "GND"
- board text removed: "Mute P"
- board text removed: "Mute R"
- board text removed: "POE+"
- board text removed: "POE-"
- board text removed: "Vol Dn"
- board text removed: "Vol Up"
Changed lines of the file:
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@@
 <circle x="37.465" y="20.955" radius="3.048" width="0.1524" layer="21"/>
 <circle x="37.465" y="-20.955" radius="3.048" width="0.1524" layer="21"/>
-<text x="-21.6" y="-10.1" size="1" layer="25" font="vector" ratio="20" align="center">Vol Up</text>
-<text x="-21.6" y="-12.3" size="1" layer="25" font="vector" ratio="20" align="center">Vol Dn</text>
-<text x="-21.6" y="-11.2" size="1" layer="25" font="vector" ratio="20" align="center">Mute P</text>
-<text x="-21.6" y="-13.4" size="1" layer="25" font="vector" ratio="20" align="center">Mute R</text>
-<text x="-30.2" y="-7.6" size="1" layer="25" font="vector" ratio="20" rot="R180" align="center">POE+</text>
-<text x="-30.2" y="-8.8" size="1" layer="25" font="vector" ratio="20" rot="R180" align="center">POE-</text>
-<text x="-30.7" y="-9.9" size="1" layer="25" font="vector" ratio="20" rot="R180" align="center">+5V</text>
-<text x="-30.7" y="-11" size="1" layer="25" font="vector" ratio="20" rot="R180" align="center">GND</text>
 </plain>
 <attributes>
@@
 <attribute name="VALUE" x="10.695" y="-9.435" size="1.27" layer="28" rot="MR90"/>
 </element>
-<element name="C14" library="pm-labs" package="0603R" value="20p" x="-12" y="-17.9" smashed="yes" rot="MR90">
-<attribute name="NAME" x="-10.9" y="-17.9" size="0.8" layer="26" font="vector" ratio="25" rot="MR90" align="center"/>
-<attribute name="VALUE" x="-13.905" y="-18.535" size="1.27" layer="28" rot="MR90"/>
-</element>
-<element name="C15" library="pm-labs" package="0603R" value="20p" x="-16.4" y="-17.9" smashed="yes" rot="MR270">
-<attribute name="NAME" x="-17.5" y="-17.9" size="0.8" layer="26" font="vector" ratio="25" rot="MR90" align="center"/>
-<attribute name="VALUE" x="-14.495" y="-17.265" size="1.27" layer="28" rot="MR270"/>
+<element name="C14" library="pm-labs" package="0603R" value="20p" x="-11.9" y="-17.9" smashed="yes" rot="MR90">
+<attribute name="NAME" x="-10.8" y="-17.9" size="0.8" layer="26" font="vector" ratio="25" rot="MR90" align="center"/>
+<attribute name="VALUE" x="-13.805" y="-18.535" size="1.27" layer="28" rot="MR90"/>
+</element>
+<element name="C15" library="pm-labs" package="0603R" value="20p" x="-16.5" y="-17.9" smashed="yes" rot="MR270">
+<attribute name="NAME" x="-17.6" y="-17.9" size="0.8" layer="26" font="vector" ratio="25" rot="MR90" align="center"/>
+<attribute name="VALUE" x="-14.595" y="-17.265" size="1.27" layer="28" rot="MR270"/>
 </element>
 <element name="C16" library="pm-labs" package="1206D-R" value="100u" x="-11.3" y="-3.4" smashed="yes" rot="MR180">
@@
 <attribute name="VALUE" x="23.63" y="-10.56" size="1.27" layer="28" rot="MR180"/>
 </element>
-<element name="C9" library="pm-labs" package="0603R" value="10u" x="-30.4" y="-10.3" smashed="yes" rot="MR270">
-<attribute name="NAME" x="-31.5" y="-10.3" size="0.8" layer="26" font="vector" ratio="25" rot="MR90" align="center"/>
-<attribute name="VALUE" x="-28.495" y="-9.665" size="1.27" layer="28" rot="MR270"/>
+<element name="C9" library="pm-labs" package="0603R" value="10u" x="-32.7" y="-10.5" smashed="yes" rot="MR270">
+<attribute name="NAME" x="-31.5" y="-9.8" size="0.8" layer="26" font="vector" ratio="25" rot="MR90" align="center"/>
+<attribute name="VALUE" x="-30.795" y="-9.865" size="1.27" layer="28" rot="MR270"/>
 </element>
 <element name="P8" library="PiProject" package="PINHEAD2X23" value="PINHEAD2X23" x="32.385" y="25.4" smashed="yes">
@@
 <wire x1="5.44" y1="17" x2="6.4" y2="17" width="0.2" layer="1"/>
 <wire x1="4.8" y1="16.36" x2="5.44" y2="17" width="0.2" layer="1"/>
-<wire x1="-30.4" y1="-9.65" x2="-30.6" y2="-9.65" width="0.5" layer="16"/>
+<wire x1="-32.7" y1="-9.85" x2="-32.9" y2="-9.85" width="0.5" layer="16"/>
 <wire x1="-38.125" y1="12.375" x2="-37.075" y2="12.375" width="0.4" layer="1"/>
 <wire x1="-37.075" y1="12.375" x2="-36.4" y2="11.7" width="0.4" layer="1"/>
@@
 <wire x1="-30.9" y1="1.75" x2="-29.95" y2="0.6" width="0.5" layer="16"/>
 <via x="-29.7" y="0.6" extent="1-16" drill="0.3"/>
-<via x="-31.63978125" y="-9.071196875" extent="1-16" drill="0.3"/>
 <wire x1="-41.45" y1="-19.2" x2="-41.3468" y2="-19.3032" width="0.2" layer="16"/>
 <wire x1="-37.9" y1="-17.5" x2="-38.7056" y2="-17.5" width="0.2" layer="16"/>
@@
 <wire x1="-39.518146875" y1="-20.331853125" x2="-39.7056" y2="-19.879303125" width="0.2" layer="16" curve="-45.00028"/>
 <wire x1="-39.7056" y1="-19.879303125" x2="-39.7056" y2="-19.3032" width="0.2" layer="16"/>
-<wire x1="-30.4" y1="-9.65" x2="-31.260978125" y2="-9.45" width="0.5" layer="16"/>
-<wire x1="-31.260978125" y1="-9.45" x2="-31.63978125" y2="-9.071196875" width="0.5" layer="16"/>
 <wire x1="8.4" y1="16.3" x2="8.4" y2="15.46" width="0.2" layer="1"/>
 <wire x1="9.274975" y1="16.4" x2="9.174975" y2="16.3" width="0.2" layer="1"/>
@@
 <wire x1="-17.6444" y1="-5.5944" x2="-18" y2="-5.5944" width="0.2" layer="16"/>
 <via x="-18" y="-5.5944" extent="1-16" drill="0.3"/>
-<wire x1="-12" y1="-17.25" x2="-13.35" y2="-17.25" width="0.2" layer="16"/>
-<wire x1="-15.05" y1="-18.55" x2="-16.4" y2="-18.55" width="0.2" layer="16"/>
-<wire x1="-16.4" y1="-18.55" x2="-16.55" y2="-18.55" width="0.2" layer="16"/>
-<wire x1="-16.55" y1="-18.55" x2="-17.2" y2="-17.9" width="0.2" layer="16"/>
-<via x="-17.2" y="-17.9" extent="1-16" drill="0.3"/>
-<wire x1="-12" y1="-17.25" x2="-11.9" y2="-17.25" width="0.2" layer="16"/>
-<via x="-11.2" y="-17.9" extent="1-16" drill="0.3"/>
-<wire x1="-12" y1="-17.25" x2="-11.85" y2="-17.25" width="0.2" layer="16"/>
-<wire x1="-11.85" y1="-17.25" x2="-11.2" y2="-17.9" width="0.2" layer="16"/>
+<wire x1="-11.9" y1="-17.25" x2="-13.35" y2="-17.25" width="0.2" layer="16"/>
+<wire x1="-15.05" y1="-18.55" x2="-16.5" y2="-18.55" width="0.2" layer="16"/>
+<wire x1="-16.5" y1="-18.55" x2="-16.65" y2="-18.55" width="0.2" layer="16"/>
+<wire x1="-16.65" y1="-18.55" x2="-17.3" y2="-17.9" width="0.2" layer="16"/>
+<via x="-17.3" y="-17.9" extent="1-16" drill="0.3"/>
+<wire x1="-11.9" y1="-17.25" x2="-11.8" y2="-17.25" width="0.2" layer="16"/>
+<via x="-11.1" y="-17.9" extent="1-16" drill="0.3"/>
+<wire x1="-11.9" y1="-17.25" x2="-11.9" y2="-17.5" width="0.2" layer="16"/>
+<wire x1="-11.5" y1="-17.9" x2="-11.9" y2="-17.5" width="0.2" layer="16"/>
+<wire x1="-11.5" y1="-17.9" x2="-11.1" y2="-17.9" width="0.2" layer="16"/>
 <wire x1="16.85" y1="-15" x2="18.05" y2="-16.2" width="0.2" layer="16"/>
 <wire x1="18.05" y1="-16.2" x2="18.8" y2="-16.2" width="0.2" layer="16"/>
@@
 <contactref element="P8" pad="2"/>
 <contactref element="P8" pad="1"/>
+<wire x1="-32.9" y1="-9.85" x2="-35.19" y2="-9.85" width="0.2" layer="16"/>
+<wire x1="-35.19" y1="-9.85" x2="-35.41" y2="-9.63" width="0.2" layer="16"/>
 </signal>
 <signal name="GPIO21">
@@
 <wire x1="-13.55" y1="-18.55" x2="-13.35" y2="-18.55" width="0.18" layer="16"/>
 <wire x1="-13.35" y1="-18.55" x2="-13.55" y2="-18.75" width="0.2" layer="16"/>
-<wire x1="-13.35" y1="-18.55" x2="-12" y2="-18.55" width="0.2" layer="16"/>
+<wire x1="-13.35" y1="-18.55" x2="-11.9" y2="-18.55" width="0.2" layer="16"/>
 </signal>
 <signal name="N$48">
@@
 <wire x1="-15.05" y1="-16.95" x2="-15.05" y2="-17.25" width="0.18" layer="16"/>
 <wire x1="-14.38" y1="-16.28" x2="-15.05" y2="-16.95" width="0.18" layer="16"/>
-<wire x1="-16.4" y1="-17.25" x2="-15.05" y2="-17.25" width="0.18" layer="16"/>
+<wire x1="-16.5" y1="-17.25" x2="-15.05" y2="-17.25" width="0.18" layer="16"/>
 </signal>
 <signal name="USB2D_P" class="1">
@@
 <wire x1="32.7" y1="-13.95" x2="32.7" y2="-12.7" width="0.5" layer="16"/>
 <wire x1="32.7" y1="-12.7" x2="33.2" y2="-12.2" width="0.5" layer="16"/>
-<wire x1="-30.4" y1="-10.95" x2="-30.95" y2="-10.95" width="0.5" layer="16"/>
-<wire x1="-30.95" y1="-10.95" x2="-32.7" y2="-12.7" width="0.5" layer="16"/>
+<wire x1="-32.7" y1="-11.15" x2="-32.7" y2="-12.7" width="0.5" layer="16"/>
 <wire x1="-14.65" y1="-5" x2="-14.65" y2="-6.2" width="0.2" layer="16"/>
 <wire x1="-14.65" y1="-6.2" x2="-14.65" y2="-6.5" width="0.2" layer="16"/>
@@
 <wire x1="-20.8" y1="-7.2" x2="-25" y2="-11.4" width="0.5" layer="1"/>
 <via x="-29.4" y="-11.4" extent="1-16" drill="0.3"/>
-<wire x1="-29.4" y1="-11.4" x2="-29.85" y2="-10.95" width="0.5" layer="16"/>
-<wire x1="-29.85" y1="-10.95" x2="-30.4" y2="-10.95" width="0.5" layer="16"/>
+<wire x1="-29.4" y1="-11.4" x2="-29.65" y2="-11.15" width="0.5" layer="16"/>
+<wire x1="-29.65" y1="-11.15" x2="-32.7" y2="-11.15" width="0.5" layer="16"/>
 <wire x1="-25" y1="-11.4" x2="-29.4" y2="-11.4" width="0.5" layer="1"/>
 <wire x1="24.4" y1="-13.1" x2="25.4" y2="-13.1" width="0.5" layer="1"/>
@@
 <contactref element="RPI-CM1" pad="153"/>
 <contactref element="U$13" pad="1"/>
-<wire x1="-31.7652125" y1="-10.3476" x2="-35.9176125" y2="-14.5" width="0.2" layer="16"/>
-<wire x1="-31.7652125" y1="-10.3476" x2="-29.59595" y2="-10.3476" width="0.2" layer="16"/>
-<wire x1="-35.9176125" y1="-14.5" x2="-36.675" y2="-14.5" width="0.2" layer="16"/>
+<wire x1="-36.675" y1="-14.5" x2="-36.675" y2="-14.0573875" width="0.2" layer="16"/>
+<wire x1="-33.1176125" y1="-10.5" x2="-36.675" y2="-14.0573875" width="0.2" layer="16"/>
+<wire x1="-33.1176125" y1="-10.5" x2="-29.44355" y2="-10.5" width="0.2" layer="16"/>
 <via x="-23.3424" y="-11" extent="1-16" drill="0.3" diameter="0.1545"/>
 <wire x1="0.4" y1="-11.7" x2="0.4" y2="-15.46" width="0.2" layer="1"/>
-<wire x1="-29.59595" y1="-10.3476" x2="-28.28795" y2="-11.6556" width="0.2" layer="16"/>
+<wire x1="-29.44355" y1="-10.5" x2="-28.28795" y2="-11.6556" width="0.2" layer="16"/>
 <wire x1="-23.3424" y1="-11" x2="-23.998" y2="-11.6556" width="0.2" layer="16"/>
 <wire x1="-23.998" y1="-11.6556" x2="-28.28795" y2="-11.6556" width="0.2" layer="16"/>

Commit message: Testing nRPIBOOT fix
Parts:
- removed !RPI_BOOT: TP1R, pm-labs:TP1R
- added Q1, Q2: BCX70SMD, transistor-npn:SOT23
Connections:
- removed net N$25: R2.A, R8.A, RPI-CM1.101, SLAVE_SWITCH.2, U$1.SEL
- removed net N$36: !RPI_BOOT.1, RPI-CM1.93
- new net !RPIBOOT: Q2.3, RPI-CM1.93
- new net N$2: LED1.C, Q1.3, R2.B
- new net N$7: Q1.2, Q2.2, SLAVE_SWITCH.2
- new net SELECT: R2.A, R8.A, RPI-CM1.101, U$1.SEL
- net +3.3V: now also Q1.1, Q2.1; no longer SLAVE_SWITCH.1
- net GND: now also SLAVE_SWITCH.1; no longer LED1.C, R2.B
Routing:
- net !RPIBOOT: track 0.00 -> 62.2 mm, vias 0 -> 3
- net SELECT: track 0.00 -> 47.6 mm, vias 0 -> 1
- net N$2: track 0.00 -> 44.0 mm
- net N$25: track 38.1 -> 0.00 mm, vias 1 -> 0
- net N$7: track 0.00 -> 12.9 mm
- net GND: track 232.5 -> 225.7 mm, vias 59 -> 60
- net N$36: track 5.92 -> 0.00 mm, vias 1 -> 0
- net +3.3V: track 58.4 -> 63.5 mm
- net USB5D_N: track 93.9 -> 94.6 mm
- net USB5D_P: track 94.5 -> 95.1 mm
- net GPIO27: track 67.2 -> 66.7 mm

Commit message: Need PM labs
replace transistor with pfet and diode with shotkey diode
Parts:
- removed Q2: BCX70SMD, transistor-npn:SOT23
- added R17: 1u, pm-labs:0603R
Connections:
- removed net N$2: LED1.C, Q1.3, R2.B
- removed net N$7: Q1.2, Q2.2, SLAVE_SWITCH.2
- new net N$8: Q1.1, R17.B, SLAVE_SWITCH.1
- net !RPIBOOT: no longer Q2.3
- net +3.3V: now also Q1.3, R17.A; no longer Q1.1, Q2.1
- net GND: now also LED1.C, R2.B, SLAVE_SWITCH.2; no longer SLAVE_SWITCH.1
- net SELECT: now also Q1.2
Routing:
- net N$2: track 44.0 -> 0.00 mm
- net GND: track 225.7 -> 261.0 mm
- net N$7: track 12.9 -> 0.00 mm
- net +3.3V: track 63.5 -> 61.4 mm
- net !RPIBOOT: track 62.2 -> 60.2 mm

Commit message: Fixed rpiboot
Parts:
- removed Q1: BCX70SMD, transistor-npn:SOT23
- added D4: PD3S160, diode:POWERDI323
- added Q2: BSS84, transistor-small-signal:SOT23
- moved R17 70.8 mm to (21.2, -16.5), flipped to the bottom, turned to 180 degrees
Connections:
- net !RPIBOOT: now also D4.A
- net +3.3V: now also Q2.2; no longer Q1.3
- net N$8: now also D4.C, Q2.1; no longer Q1.1
- net SELECT: now also Q2.3; no longer Q1.2
Routing:
- net GND: track 261.0 -> 231.5 mm
- net N$8: track 0.00 -> 14.5 mm
- net SELECT: track 47.6 -> 61.2 mm
- net !RPIBOOT: track 60.2 -> 62.4 mm
- net +3.3V: track 61.4 -> 59.9 mm, vias 10 -> 11

Commit message: Fixed RPI and USB switch Pulldown
Parts:
- moved D4 0.80 mm to (20.7, -17.9)
Routing:
- net N$8: track 14.5 -> 15.3 mm
Changed lines of the file:
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@@
 <attribute name="VALUE" x="19.9" y="-16.5" size="1.27" layer="28" font="vector" rot="MR270" align="bottom-center"/>
 </element>
-<element name="D4" library="diode" library_urn="urn:adsk.eagle:library:210" package="POWERDI323" package3d_urn="urn:adsk.eagle:package:43459/1" value="PD3S160" x="21.5" y="-17.9" smashed="yes" rot="MR0">
-<attribute name="NAME" x="10.3214" y="-21.9484" size="1.27" layer="26" rot="MR270"/>
-<attribute name="POPULARITY" value="0" x="21.5" y="-17.9" size="1.778" layer="28" rot="MR0" display="off"/>
-<attribute name="VALUE" x="23.3516" y="-20.4566" size="1.27" layer="28" rot="MR0"/>
+<element name="D4" library="diode" library_urn="urn:adsk.eagle:library:210" package="POWERDI323" package3d_urn="urn:adsk.eagle:package:43459/1" value="PD3S160" x="20.7" y="-17.9" smashed="yes" rot="MR0">
+<attribute name="NAME" x="9.5214" y="-21.9484" size="1.27" layer="26" rot="MR270"/>
+<attribute name="POPULARITY" value="0" x="20.7" y="-17.9" size="1.778" layer="28" rot="MR0" display="off"/>
+<attribute name="VALUE" x="22.5516" y="-20.4566" size="1.27" layer="28" rot="MR0"/>
 </element>
 <element name="Q2" library="transistor-small-signal" library_urn="urn:adsk.eagle:library:401" package="SOT23" package3d_urn="urn:adsk.eagle:package:28738/2" value="BSS84" x="24.1" y="-17.3" smashed="yes" rot="MR180">
@@
 <wire x1="-9.986025" y1="15.386025" x2="-9.986025" y2="13.554275" width="0.2" layer="16"/>
 <contactref element="D4" pad="A"/>
-<wire x1="20.35" y1="-17.9" x2="19.5" y2="-17.05" width="0.2" layer="16"/>
-<wire x1="19.5" y1="-17.05" x2="19.5" y2="-16.9" width="0.2" layer="16"/>
+<wire x1="19.55" y1="-17.9" x2="19.5" y2="-17.85" width="0.2" layer="16"/>
+<wire x1="19.5" y1="-17.85" x2="19.5" y2="-16.9" width="0.2" layer="16"/>
 </signal>
 <signal name="N$38">
@@
 <wire x1="24.1" y1="-18.4" x2="23.65695" y2="-18.4" width="0.2" layer="16"/>
 <wire x1="23.65695" y1="-18.4" x2="23.35455" y2="-18.7024" width="0.2" layer="16"/>
-<wire x1="23.35455" y1="-18.7024" x2="19.99545" y2="-18.7024" width="0.2" layer="16"/>
-<wire x1="19.99545" y1="-18.7024" x2="17.79305" y2="-16.5" width="0.2" layer="16"/>
+<wire x1="23.35455" y1="-18.7024" x2="19.19545" y2="-18.7024" width="0.2" layer="16"/>
+<wire x1="19.19545" y1="-18.7024" x2="16.99305" y2="-16.5" width="0.2" layer="16"/>
 <wire x1="13.1" y1="-16.5" x2="11.8" y2="-15.2" width="0.2" layer="16"/>
-<wire x1="17.79305" y1="-16.5" x2="13.1" y2="-16.5" width="0.2" layer="16"/>
+<wire x1="16.99305" y1="-16.5" x2="13.1" y2="-16.5" width="0.2" layer="16"/>
 </signal>
 <signal name="N$8">
@@
 <wire x1="21.85" y1="-16.5" x2="22.15" y2="-16.2" width="0.2" layer="16"/>
 <wire x1="22.15" y1="-16.2" x2="23.15" y2="-16.2" width="0.2" layer="16"/>
-<wire x1="22.25" y1="-17.9" x2="22.85" y2="-17.3" width="0.2" layer="16"/>
+<wire x1="21.45" y1="-17.9" x2="22.05" y2="-17.3" width="0.2" layer="16"/>
 <wire x1="25.63703125" y1="-17.3" x2="26.72003125" y2="-18.383" width="0.2" layer="16"/>
 <wire x1="26.72003125" y1="-18.383" x2="28.27996875" y2="-18.383" width="0.2" layer="16"/>
 <wire x1="28.27996875" y1="-18.383" x2="29.22296875" y2="-17.44" width="0.2" layer="16"/>
 <wire x1="29.22296875" y1="-17.44" x2="32.72" y2="-17.44" width="0.2" layer="16"/>
-<wire x1="22.85" y1="-17.3" x2="24.25" y2="-17.3" width="0.2" layer="16"/>
+<wire x1="22.05" y1="-17.3" x2="24.25" y2="-17.3" width="0.2" layer="16"/>
 <wire x1="23.15" y1="-16.2" x2="24.25" y2="-17.3" width="0.2" layer="16"/>
 <wire x1="24.25" y1="-17.3" x2="25.63703125" y2="-17.3" width="0.2" layer="16"/>

Commit message: minor fixes
Routing:
- net POE+: track 34.2 -> 32.6 mm
- net GND: track 231.5 -> 230.0 mm
