File: CarrierBoard/PiProjector.brd (EAGLE design)
At the start: 86.4 x 54.6 mm, 74 parts, among them P8 PINHEAD2X23, P9 PINHEAD2X23, Q2 BSS84, X1 24MHz, X2 12Mhz

Commit message: Added an I2C expander
Connections:
- net GPIO23 renamed SDA
- net GPIO24 renamed SCL
Changed lines of the file:
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@@
 <wire x1="2.8" y1="-14.2" x2="2.4" y2="-14.6" width="0.2" layer="1"/>
 </signal>
-<signal name="GPIO23">
+<signal name="SDA">
 <contactref element="P9" pad="20"/>
 <contactref element="RPI-CM1" pad="47"/>
@@
 <wire x1="1.5" y1="-15.7" x2="1.7" y2="-15.9" width="0.2" layer="16"/>
 </signal>
-<signal name="GPIO24">
+<signal name="SCL">
 <contactref element="P9" pad="19"/>
 <contactref element="RPI-CM1" pad="45"/>

Commit message: forgot to push last version after sending to OSH
Parts:
- added +3.3V, +5V, ACT_LED, GND, PWR_LED: TP1R, pm-labs:TP1R
- R17: value 1u -> 10K
- moved GLOBAL_EN 0.41 mm to (-11.1, 17.0)
Connections:
- new net N$1: PWR_LED.1, RPI-CM1.95
- new net N$2: ACT_LED.1, RPI-CM1.21
- net +3.3V: now also +3.3V.1
- net +5V: now also +5V.1
- net GND: now also GND.1
Routing:
- net N$1: track 0.00 -> 4.69 mm, vias 0 -> 1
- net SELECT: track 61.2 -> 57.3 mm
- net N$2: track 0.00 -> 2.88 mm, vias 0 -> 1
- net POE-: track 40.7 -> 41.9 mm
- net +3.3V: track 59.9 -> 61.0 mm, vias 11 -> 12
- net +5V: track 66.7 -> 67.7 mm, vias 6 -> 7
- net GND: track 230.0 -> 231.0 mm, vias 60 -> 61
- net POE+: track 32.6 -> 31.8 mm
- net LEDG: track 45.1 -> 45.9 mm
- net PAIR1_N: track 51.2 -> 50.4 mm
- net PAIR1_P: track 46.2 -> 45.4 mm
- net PAIR0_N: track 45.5 -> 44.7 mm
- net PAIR0_P: track 41.5 -> 40.8 mm
- net N$21: track 39.1 -> 39.8 mm
Other:
- board text added: "1"
- board text added: "PI_CO_PROJECTOR Rev 2.0 - MAIN JAKUB NEJEDLY"

Commit message: Modified POE route  to avoid clearence issues
Routing:
- net N$43: track 10.9 -> 9.53 mm, vias 0 -> 1
- net N$33: track 7.73 -> 8.98 mm, vias 0 -> 1
- net POE-: track 41.9 -> 42.6 mm
Changed lines of the file:
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@@
 <layer number="13" name="Route13" color="21" fill="1" visible="no" active="no"/>
 <layer number="14" name="Route14" color="22" fill="1" visible="no" active="no"/>
-<layer number="15" name="Route15" color="23" fill="1" visible="yes" active="yes"/>
+<layer number="15" name="Route15" color="23" fill="1" visible="no" active="yes"/>
 <layer number="16" name="Bottom" color="1" fill="1" visible="yes" active="yes"/>
 <layer number="17" name="Pads" color="2" fill="1" visible="yes" active="yes"/>
@@
 <wire x1="-37.125" y1="5.375" x2="-37.1" y2="5.4" width="0.5" layer="16"/>
 <contactref element="P8" pad="6"/>
-<wire x1="-37.6" y1="5.4" x2="-37.1" y2="5.4" width="0.5" layer="1"/>
-<wire x1="-37.9" y1="1.5" x2="-37.6" y2="1.8" width="0.5" layer="1"/>
-<wire x1="-37.6" y1="5.4" x2="-37.6" y2="1.8" width="0.5" layer="1"/>
+<wire x1="-37.1" y1="5.4" x2="-37.6" y2="5.4" width="0.5" layer="1"/>
 <wire x1="-34.86303125" y1="11.8654" x2="-37.603" y2="9.12543125" width="0.5" layer="1"/>
 <wire x1="-37.603" y1="9.12543125" x2="-37.603" y2="5.4" width="0.5" layer="1"/>
@@
 <wire x1="-30.4" y1="11.3654" x2="-30.9" y2="11.8654" width="0.5" layer="1" curve="90"/>
 <wire x1="-30.9" y1="11.8654" x2="-34.86303125" y2="11.8654" width="0.5" layer="1"/>
+<wire x1="-37.9" y1="2.13141875" x2="-37.9" y2="1.5" width="0.5" layer="1"/>
+<wire x1="-38.7556" y1="2.98701875" x2="-37.9" y2="2.13141875" width="0.5" layer="1"/>
+<wire x1="-37.6" y1="5.4" x2="-38.7556" y2="4.2444" width="0.5" layer="1"/>
+<wire x1="-38.7556" y1="4.2444" x2="-38.7556" y2="2.98701875" width="0.5" layer="1"/>
 </signal>
 <signal name="N$37">
@@
 <contactref element="D1" pad="3"/>
 <contactref element="U$5" pad="11"/>
-<wire x1="-31.72474375" y1="8.128" x2="-31.365" y2="8.128" width="0.5" layer="16"/>
-<wire x1="-37.85" y1="3.35" x2="-37.125" y2="3.35" width="0.5" layer="16"/>
-<wire x1="-37.85" y1="3.35" x2="-37.9" y2="3.4" width="0.5" layer="16"/>
-<wire x1="-37.9" y1="5.66858125" x2="-37.41298125" y2="6.1556" width="0.5" layer="16"/>
-<wire x1="-37.41298125" y1="6.1556" x2="-36.72803125" y2="6.1556" width="0.5" layer="16"/>
-<wire x1="-36.72803125" y1="6.1556" x2="-36.39243125" y2="5.82" width="0.5" layer="16"/>
-<wire x1="-37.9" y1="3.4" x2="-37.9" y2="5.66858125" width="0.5" layer="16"/>
-<wire x1="-36.39243125" y1="5.82" x2="-34.03274375" y2="5.82" width="0.5" layer="16"/>
-<wire x1="-34.03274375" y1="5.82" x2="-31.72474375" y2="8.128" width="0.5" layer="16"/>
+<via x="-38" y="3.3" extent="1-16" drill="0.3"/>
+<wire x1="-31.365" y1="8.128" x2="-32.7526" y2="6.7404" width="0.5" layer="1"/>
+<wire x1="-32.7526" y1="6.7404" x2="-33.11234375" y2="6.7404" width="0.5" layer="1"/>
+<wire x1="-36.55274375" y1="3.3" x2="-38" y2="3.3" width="0.5" layer="1"/>
+<wire x1="-33.11234375" y1="6.7404" x2="-36.55274375" y2="3.3" width="0.5" layer="1"/>
+<wire x1="-38" y1="3.3" x2="-37.95" y2="3.35" width="0.5" layer="16"/>
+<wire x1="-37.95" y1="3.35" x2="-37.125" y2="3.35" width="0.5" layer="16"/>
 </signal>
 <signal name="N$33">
 <contactref element="D2" pad="3"/>
 <contactref element="U$5" pad="14"/>
-<wire x1="-37.125" y1="0.15" x2="-37.125" y2="-0.775" width="0.5" layer="16"/>
-<wire x1="-37.125" y1="-0.775" x2="-36.9" y2="-1" width="0.5" layer="16"/>
-<wire x1="-36.9" y1="-1" x2="-34.09156875" y2="-1" width="0.5" layer="16"/>
-<wire x1="-31.78956875" y1="-3.302" x2="-31.365" y2="-3.302" width="0.5" layer="16"/>
-<wire x1="-34.09156875" y1="-1" x2="-31.78956875" y2="-3.302" width="0.5" layer="16"/>
+<wire x1="-37.125" y1="0.15" x2="-37.95" y2="0.15" width="0.5" layer="16"/>
+<wire x1="-37.95" y1="0.15" x2="-38" y2="0.2" width="0.5" layer="16"/>
+<via x="-38" y="0.2" extent="1-16" drill="0.3"/>
+<wire x1="-33.11234375" y1="-1.9144" x2="-32.7526" y2="-1.9144" width="0.5" layer="1"/>
+<wire x1="-32.7526" y1="-1.9144" x2="-31.365" y2="-3.302" width="0.5" layer="1"/>
+<wire x1="-38" y1="0.2" x2="-35.22674375" y2="0.2" width="0.5" layer="1"/>
+<wire x1="-35.22674375" y1="0.2" x2="-33.11234375" y2="-1.9144" width="0.5" layer="1"/>
 </signal>
 <signal name="N$34">

Commit message: Added images and Rerouted POE
Routing:
- net +3.3V: track 61.0 -> 59.8 mm
- net GND: track 231.0 -> 230.1 mm
Changed lines of the file:
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@@
 <wire x1="28.2" y1="-12.2112" x2="28.2" y2="-12.72085" width="0.2" layer="16"/>
 <wire x1="28.2" y1="-12.72085" x2="27.6" y2="-13.32085" width="0.2" layer="16"/>
-<via x="26.4588" y="-7.5" extent="1-16" drill="0.3"/>
-<wire x1="25.34915" y1="-7.9056" x2="25.85085" y2="-7.9056" width="0.2" layer="16"/>
-<wire x1="24.65" y1="-7.5" x2="24.94355" y2="-7.5" width="0.2" layer="16"/>
-<wire x1="26.25645" y1="-7.5" x2="26.4588" y2="-7.5" width="0.2" layer="16"/>
-<wire x1="24.94355" y1="-7.5" x2="25.34915" y2="-7.9056" width="0.2" layer="16"/>
-<wire x1="25.85085" y1="-7.9056" x2="26.25645" y2="-7.5" width="0.2" layer="16"/>
-<wire x1="26.8" y1="-5.65" x2="26.8" y2="-7.1588" width="0.2" layer="16"/>
-<wire x1="26.8" y1="-7.1588" x2="26.4588" y2="-7.5" width="0.2" layer="16"/>
 <via x="18.8" y="-16.2" extent="1-16" drill="0.3"/>
 <wire x1="-33.65" y1="22.32" x2="-33.05" y2="21.72" width="0.2" layer="16"/>
@@
 <wire x1="-10.7" y1="15.4" x2="-11.1" y2="15" width="0.2" layer="16"/>
 <via x="-10.7" y="15.9" extent="1-16" drill="0.3"/>
+<wire x1="26.8" y1="-5.65" x2="26.8" y2="-6.3" width="0.2" layer="16"/>
+<wire x1="26.8" y1="-6.3" x2="25.6" y2="-7.5" width="0.2" layer="16"/>
+<via x="25.6" y="-7.5" extent="1-16" drill="0.3"/>
+<wire x1="24.65" y1="-7.5" x2="25.6" y2="-7.5" width="0.2" layer="16"/>
 </signal>
 <signal name="GPIO21">
@@
 <wire x1="26.55" y1="-11.5" x2="26.63235" y2="-11.5" width="0.2" layer="16"/>
 <wire x1="27.5944" y1="-12.46205" x2="26.63235" y2="-11.5" width="0.2" layer="16"/>
-<wire x1="22.11" y1="-8.09" x2="22.7" y2="-7.5" width="0.2" layer="16"/>
-<wire x1="22.7" y1="-7.5" x2="23.35" y2="-7.5" width="0.2" layer="16"/>
-<via x="25.6" y="-7.3" extent="1-16" drill="0.3"/>
-<wire x1="24.24670625" y1="-6.8476" x2="25.05329375" y2="-6.8476" width="0.2" layer="16"/>
+<wire x1="22.7" y1="-7.5" x2="22.11" y2="-8.09" width="0.2" layer="16"/>
+<via x="22.9" y="-6.4" extent="1-16" drill="0.3"/>
 <wire x1="23.35" y1="-7.5" x2="23.59430625" y2="-7.5" width="0.2" layer="16"/>
-<wire x1="23.59430625" y1="-7.5" x2="24.24670625" y2="-6.8476" width="0.2" layer="16"/>
-<wire x1="25.50569375" y1="-7.3" x2="25.6" y2="-7.3" width="0.2" layer="16"/>
-<wire x1="25.05329375" y1="-6.8476" x2="25.50569375" y2="-7.3" width="0.2" layer="16"/>
 <wire x1="16.71" y1="-8.09" x2="16.6" y2="-7.98" width="0.2" layer="16"/>
 <wire x1="16.6" y1="-7.98" x2="16.6" y2="-6.15" width="0.2" layer="16"/>
@@
 <wire x1="-10.7" y1="13.9944" x2="-10.7" y2="13.5" width="0.2" layer="16"/>
 <via x="-10.7" y="13.9944" extent="1-16" drill="0.3"/>
+<wire x1="23.35" y1="-7.5" x2="22.7" y2="-7.5" width="0.2" layer="16"/>
+<wire x1="23.35" y1="-7.5" x2="23.35" y2="-6.85" width="0.2" layer="16"/>
+<wire x1="23.35" y1="-6.85" x2="22.9" y2="-6.4" width="0.2" layer="16"/>
 </signal>
 <signal name="+5V" class="3">
