File: CarrierBoard/PiProjector.sch (EAGLE design)
At the start: 73 parts, among them P8 PINHEAD2X23, P9 PINHEAD2X23, Q1 BCX70SMD, X1 24MHz, X2 12Mhz

Commit message: Fixed rpiboot
Parts:
- removed Q1: BCX70SMD, transistor-npn:BCX70SMD
- added D4: PD3S160, diode:PD3S160
- added Q2: BSS84, transistor-small-signal:BSS84
Connections:
- net !RPIBOOT: now also D4.A
- net +3.3V: now also Q2.S; no longer Q1.C
- net N$8: now also D4.C, Q2.G; no longer Q1.B
- net SELECT: now also Q2.D; no longer Q1.E
Other:
- moved on the sheet: R17
Changed lines of the file:
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@@
 <part name="SUPPLY29" library="supply2" library_urn="urn:adsk.eagle:library:372" deviceset="GND" device=""/>
 <part name="SUPPLY30" library="supply2" library_urn="urn:adsk.eagle:library:372" deviceset="GND" device=""/>
-<part name="Q1" library="transistor-npn" library_urn="urn:adsk.eagle:library:398" deviceset="BCX70*" device="SMD" package3d_urn="urn:adsk.eagle:package:28738/2"/>
 <part name="R17" library="pm-labs" deviceset="R" device="0603R" value="1u"/>
 <part name="SUPPLY5" library="supply2" library_urn="urn:adsk.eagle:library:372" deviceset="GND" device=""/>
 <part name="SUPPLY22" library="supply2" library_urn="urn:adsk.eagle:library:372" deviceset="GND" device=""/>
-<part name="D3" library="docu-dummy" library_urn="urn:adsk.eagle:library:215" deviceset="DIODE" device=""/>
+<part name="D4" library="diode" library_urn="urn:adsk.eagle:library:210" deviceset="PD3S160" device="" package3d_urn="urn:adsk.eagle:package:43459/1"/>
+<part name="Q2" library="transistor-small-signal" library_urn="urn:adsk.eagle:library:401" deviceset="BSS84" device="" package3d_urn="urn:adsk.eagle:package:28738/2"/>
 </parts>
 <sheets>
@@
 <attribute name="VALUE" x="-45.085" y="210.185" size="1.778" layer="96"/>
 </instance>
-<instance part="Q1" gate="G$1" x="147.32" y="195.58" smashed="yes">
-<attribute name="NAME" x="144.78" y="193.04" size="1.778" layer="95" rot="R180"/>
-</instance>
-<instance part="R17" gate="R" x="142.24" y="203.2" smashed="yes" rot="R270">
-<attribute name="NAME" x="144.78" y="208.28" size="1.778" layer="95" rot="R270"/>
-<attribute name="VALUE" x="144.78" y="203.2" size="1.778" layer="96" rot="R270"/>
+<instance part="R17" gate="R" x="142.24" y="205.74" smashed="yes" rot="R270">
+<attribute name="NAME" x="144.78" y="210.82" size="1.778" layer="95" rot="R270"/>
+<attribute name="VALUE" x="144.78" y="205.74" size="1.778" layer="96" rot="R270"/>
 </instance>
 <instance part="SUPPLY5" gate="GND" x="162.56" y="157.48" smashed="yes">
@@
 <attribute name="VALUE" x="137.795" y="154.305" size="1.778" layer="96"/>
 </instance>
-<instance part="D3" gate="G$1" x="139.7" y="200.66" smashed="yes" rot="R270"/>
+<instance part="D4" gate="G$1" x="139.7" y="203.2" smashed="yes" rot="R270">
+<attribute name="NAME" x="141.605" y="205.486" size="1.778" layer="95" rot="R270"/>
+<attribute name="VALUE" x="136.271" y="205.486" size="1.778" layer="96" rot="R270"/>
+</instance>
+<instance part="Q2" gate="G$1" x="149.86" y="195.58" smashed="yes">
+<attribute name="NAME" x="152.4" y="195.58" size="1.778" layer="95"/>
+<attribute name="VALUE" x="152.4" y="193.04" size="1.778" layer="96"/>
+</instance>
 </instances>
 <busses>
@@
 </segment>
 <segment>
-<pinref part="Q1" gate="G$1" pin="C"/>
-<wire x1="149.86" y1="208.28" x2="149.86" y2="200.66" width="0.1524" layer="91"/>
+<wire x1="149.86" y1="210.82" x2="149.86" y2="200.66" width="0.1524" layer="91"/>
 <pinref part="R17" gate="R" pin="1"/>
-<wire x1="149.86" y1="208.28" x2="142.24" y2="208.28" width="0.1524" layer="91"/>
-<junction x="149.86" y="208.28"/>
-<wire x1="149.86" y1="213.36" x2="149.86" y2="208.28" width="0.1524" layer="91"/>
+<wire x1="149.86" y1="210.82" x2="142.24" y2="210.82" width="0.1524" layer="91"/>
+<junction x="149.86" y="210.82"/>
 <label x="149.86" y="210.82" size="1.778" layer="95" rot="R90"/>
+<pinref part="Q2" gate="G$1" pin="S"/>
+<wire x1="149.86" y1="210.82" x2="149.86" y2="218.44" width="0.1524" layer="91"/>
 </segment>
 </net>
@@
 </segment>
 <segment>
-<wire x1="139.7" y1="203.2" x2="139.7" y2="213.36" width="0.1524" layer="91"/>
-<label x="139.7" y="203.2" size="1.778" layer="95" rot="R90"/>
+<wire x1="139.7" y1="205.74" x2="139.7" y2="213.36" width="0.1524" layer="91"/>
+<label x="139.7" y="205.74" size="1.778" layer="95" rot="R90"/>
+<pinref part="D4" gate="G$1" pin="A"/>
 </segment>
 </net>
@@
 <wire x1="157.48" y1="195.58" x2="157.48" y2="187.96" width="0.1524" layer="91"/>
 <label x="157.48" y="190.5" size="1.778" layer="95" rot="R90"/>
-<pinref part="Q1" gate="G$1" pin="E"/>
 <wire x1="157.48" y1="187.96" x2="157.48" y2="177.8" width="0.1524" layer="91"/>
 <wire x1="149.86" y1="190.5" x2="149.86" y2="187.96" width="0.1524" layer="91"/>
 <wire x1="149.86" y1="187.96" x2="157.48" y2="187.96" width="0.1524" layer="91"/>
 <junction x="157.48" y="187.96"/>
+<pinref part="Q2" gate="G$1" pin="D"/>
 </segment>
 </net>
@@
 <segment>
 <pinref part="R17" gate="R" pin="2"/>
-<wire x1="142.24" y1="198.12" x2="142.24" y2="195.58" width="0.1524" layer="91"/>
-<pinref part="Q1" gate="G$1" pin="B"/>
-<wire x1="142.24" y1="195.58" x2="144.78" y2="195.58" width="0.1524" layer="91"/>
-<wire x1="142.24" y1="195.58" x2="139.7" y2="195.58" width="0.1524" layer="91"/>
-<wire x1="139.7" y1="195.58" x2="139.7" y2="185.42" width="0.1524" layer="91"/>
-<junction x="142.24" y="195.58"/>
+<wire x1="142.24" y1="200.66" x2="142.24" y2="198.12" width="0.1524" layer="91"/>
+<wire x1="142.24" y1="198.12" x2="144.78" y2="198.12" width="0.1524" layer="91"/>
+<wire x1="142.24" y1="198.12" x2="139.7" y2="198.12" width="0.1524" layer="91"/>
+<wire x1="139.7" y1="198.12" x2="139.7" y2="185.42" width="0.1524" layer="91"/>
+<junction x="142.24" y="198.12"/>
 <pinref part="SLAVE_SWITCH" gate="G$1" pin="1"/>
-<wire x1="139.7" y1="195.58" x2="139.7" y2="198.12" width="0.1524" layer="91"/>
-<junction x="139.7" y="195.58"/>
-</segment>
-</net>
+<wire x1="139.7" y1="198.12" x2="139.7" y2="200.66" width="0.1524" layer="91"/>
+<junction x="139.7" y="198.12"/>
+<pinref part="D4" gate="G$1" pin="C"/>
+<pinref part="Q2" gate="G$1" pin="G"/>
+</segment>
+</net>

Commit message: Fixed RPI and USB switch Pulldown
Changed lines of the file:
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@@
 <wire x1="157.48" y1="195.58" x2="162.56" y2="195.58" width="0.1524" layer="91"/>
 <wire x1="157.48" y1="195.58" x2="157.48" y2="187.96" width="0.1524" layer="91"/>
-<label x="157.48" y="190.5" size="1.778" layer="95" rot="R90"/>
 <wire x1="157.48" y1="187.96" x2="157.48" y2="177.8" width="0.1524" layer="91"/>
 <wire x1="149.86" y1="190.5" x2="149.86" y2="187.96" width="0.1524" layer="91"/>

Commit message: Added an I2C expander
Connections:
- net GPIO23 renamed SDA
- net GPIO24 renamed SCL
Changed lines of the file:
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@@
 </segment>
 </net>
-<net name="GPIO23" class="0">
+<net name="SDA" class="0">
 <segment>
 <pinref part="P9" gate="G$1" pin="20"/>
@@
 </segment>
 </net>
-<net name="GPIO24" class="0">
+<net name="SCL" class="0">
 <segment>
 <pinref part="P9" gate="G$1" pin="19"/>

Commit message: forgot to push last version after sending to OSH
Parts:
- added +3.3V, +5V, ACT_LED, GND, PWR_LED: TP1R, pm-labs:TP1R
- R17: value 1u -> 10K
Connections:
- new net N$1: PWR_LED.1, RPI-CM1G$1.PI_LED_!PWR
- new net N$2: ACT_LED.1, RPI-CM1G$1.PI_!LED_ACTIVITY
- net +3.3V: now also +3.3V.1
- net +5V: now also +5V.1
- net GND: now also GND.1
Other:
- moved on the sheet: GLOBAL_EN
Changed lines of the file:
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@@
 <layer number="3" name="Route3" color="17" fill="1" visible="no" active="no"/>
 <layer number="4" name="Route4" color="18" fill="1" visible="no" active="no"/>
-<layer number="5" name="Route5" color="19" fill="1" visible="no" active="no"/>
+<layer number="5" name="Route5" color="4" fill="4" visible="no" active="no"/>
 <layer number="6" name="Route6" color="25" fill="1" visible="no" active="no"/>
 <layer number="7" name="Route7" color="26" fill="1" visible="no" active="no"/>
@@
 <part name="SUPPLY29" library="supply2" library_urn="urn:adsk.eagle:library:372" deviceset="GND" device=""/>
 <part name="SUPPLY30" library="supply2" library_urn="urn:adsk.eagle:library:372" deviceset="GND" device=""/>
-<part name="R17" library="pm-labs" deviceset="R" device="0603R" value="1u"/>
+<part name="R17" library="pm-labs" deviceset="R" device="0603R" value="10K"/>
 <part name="SUPPLY5" library="supply2" library_urn="urn:adsk.eagle:library:372" deviceset="GND" device=""/>
 <part name="SUPPLY22" library="supply2" library_urn="urn:adsk.eagle:library:372" deviceset="GND" device=""/>
 <part name="D4" library="diode" library_urn="urn:adsk.eagle:library:210" deviceset="PD3S160" device="" package3d_urn="urn:adsk.eagle:package:43459/1"/>
 <part name="Q2" library="transistor-small-signal" library_urn="urn:adsk.eagle:library:401" deviceset="BSS84" device="" package3d_urn="urn:adsk.eagle:package:28738/2"/>
+<part name="PWR_LED" library="pm-labs" deviceset="TP" device="1R"/>
+<part name="+5V" library="pm-labs" deviceset="TP" device="1R"/>
+<part name="+3.3V" library="pm-labs" deviceset="TP" device="1R"/>
+<part name="GND" library="pm-labs" deviceset="TP" device="1R"/>
+<part name="ACT_LED" library="pm-labs" deviceset="TP" device="1R"/>
 </parts>
 <sheets>
@@
 <attribute name="VALUE" x="175.641" y="201.676" size="1.778" layer="96" rot="R270"/>
 </instance>
-<instance part="GLOBAL_EN" gate="G" x="-15.24" y="2.54" smashed="yes" rot="R90">
-<attribute name="NAME" x="-19.05" y="2.54" size="1.27" layer="95" rot="R180" align="center-left"/>
+<instance part="GLOBAL_EN" gate="G" x="-17.78" y="2.54" smashed="yes" rot="R90">
+<attribute name="NAME" x="-21.59" y="2.54" size="1.27" layer="95" rot="R180" align="center-left"/>
 </instance>
 <instance part="U$15" gate="G$1" x="279.4" y="78.74" smashed="yes" rot="R180"/>
@@
 <attribute name="NAME" x="152.4" y="195.58" size="1.778" layer="95"/>
 <attribute name="VALUE" x="152.4" y="193.04" size="1.778" layer="96"/>
+</instance>
+<instance part="PWR_LED" gate="G" x="-17.78" y="7.62" smashed="yes" rot="R90">
+<attribute name="NAME" x="-21.59" y="7.62" size="1.27" layer="95" rot="R180" align="center-left"/>
+</instance>
+<instance part="+5V" gate="G" x="-17.78" y="15.24" smashed="yes" rot="R90">
+<attribute name="NAME" x="-21.59" y="15.24" size="1.27" layer="95" rot="R180" align="center-left"/>
+</instance>
+<instance part="+3.3V" gate="G" x="-17.78" y="30.48" smashed="yes">
+<attribute name="NAME" x="-17.78" y="34.29" size="1.27" layer="95" rot="R90" align="center-left"/>
+</instance>
+<instance part="GND" gate="G" x="-10.16" y="-2.54" smashed="yes" rot="R90">
+<attribute name="NAME" x="-13.97" y="-2.54" size="1.27" layer="95" rot="R180" align="center-left"/>
+</instance>
+<instance part="ACT_LED" gate="G" x="-12.7" y="101.6" smashed="yes" rot="R90">
+<attribute name="NAME" x="-8.89" y="104.14" size="1.27" layer="95" rot="R180" align="center-left"/>
 </instance>
 </instances>
@@
 <wire x1="-5.08" y1="60.96" x2="-7.62" y2="60.96" width="0.1524" layer="91"/>
 <junction x="-7.62" y="60.96"/>
+<pinref part="GND" gate="G" pin="1"/>
+<junction x="-7.62" y="-2.54"/>
 </segment>
 <segment>
@@
 <junction x="-33.02" y="27.94"/>
 <label x="-25.4" y="27.94" size="1.778" layer="95"/>
+<pinref part="+3.3V" gate="G" pin="1"/>
 </segment>
 <segment>
@@
 <wire x1="-5.08" y1="27.94" x2="-10.16" y2="27.94" width="0.1524" layer="91"/>
 <junction x="-10.16" y="27.94"/>
-<wire x1="-10.16" y1="17.78" x2="-10.16" y2="7.62" width="0.1524" layer="91"/>
+<wire x1="-10.16" y1="17.78" x2="-10.16" y2="15.24" width="0.1524" layer="91"/>
 <junction x="-10.16" y="17.78"/>
-<label x="-10.16" y="7.62" size="1.778" layer="95" rot="R90"/>
+<label x="-15.24" y="15.24" size="1.778" layer="95"/>
+<wire x1="-10.16" y1="15.24" x2="-15.24" y2="15.24" width="0.1524" layer="91"/>
+<pinref part="+5V" gate="G" pin="1"/>
 </segment>
 <segment>
@@
 <pinref part="GLOBAL_EN" gate="G" pin="1"/>
 <pinref part="RPI-CM1" gate="G$1" pin="GLOBAL_EN"/>
-<wire x1="-12.7" y1="2.54" x2="-5.08" y2="2.54" width="0.1524" layer="91"/>
+<wire x1="-15.24" y1="2.54" x2="-5.08" y2="2.54" width="0.1524" layer="91"/>
 </segment>
 </net>
@@
 </segment>
 </net>
+<net name="N$1" class="0">
+<segment>
+<pinref part="PWR_LED" gate="G" pin="1"/>
+<pinref part="RPI-CM1" gate="G$1" pin="PI_LED_!PWR"/>
+<wire x1="-15.24" y1="7.62" x2="-5.08" y2="7.62" width="0.1524" layer="91"/>
+</segment>
+</net>
+<net name="N$2" class="0">
+<segment>
+<pinref part="RPI-CM1" gate="G$1" pin="PI_!LED_ACTIVITY"/>
+<pinref part="ACT_LED" gate="G" pin="1"/>
+<wire x1="-10.16" y1="101.6" x2="-5.08" y2="101.6" width="0.1524" layer="91"/>
+</segment>
+</net>
