File: DaughterBoard/DaughterBoard.sch (EAGLE design)
At the start: 6 parts

Commit message: Finished modified daughterboard
Parts:
- added JP2: (no value), pinhead:PINHD-2X8
- JP1: device pinhead:PINHD-2X4 -> pinhead:PINHD-2X8
Connections:
- net +5V: now also JP1.13, JP1.14; no longer JP1.4
- net GND: now also JP1.15, JP1.16; no longer JP1.2
- net MUTP: now also JP1.10, U$5.3, U$5.4; no longer JP1.5, U$4.3, U$4.4
- net MUTR: now also JP1.9, U$3.3, U$3.4; no longer JP1.1, U$2.3, U$2.4
- net POE+: now also JP1.12; no longer JP1.8
- net POE-: now also JP1.11; no longer JP1.6
- net VLDN: now also JP1.7, U$2.3, U$2.4; no longer JP1.3, U$3.3, U$3.4
- net VLUP: now also JP1.8, U$4.3, U$4.4; no longer JP1.7, U$5.3, U$5.4

Commit message: minor fix
Other:
- moved on the sheet: JP2
Changed lines of the file:
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@@
 <attribute name="VALUE" x="-1.27" y="17.78" size="1.778" layer="96"/>
 </instance>
-<instance part="JP2" gate="A" x="96.52" y="35.56" smashed="yes">
-<attribute name="NAME" x="90.17" y="46.355" size="1.778" layer="95"/>
-<attribute name="VALUE" x="90.17" y="20.32" size="1.778" layer="96"/>
+<instance part="JP2" gate="A" x="53.34" y="33.02" smashed="yes">
+<attribute name="NAME" x="46.99" y="43.815" size="1.778" layer="95"/>
+<attribute name="VALUE" x="46.99" y="17.78" size="1.778" layer="96"/>
 </instance>
 <instance part="SUPPLY1" gate="GND" x="5.08" y="-20.32" smashed="yes">

Commit message: Added an I2C expander
Parts:
- added U$6: GPIOEX_TCA9539PWR, PicoDaughterBoard:GPIOEX_TCA9539PWR
- added U$7, U$8: BTN-222CJVABR, PicoDaughterBoard:BTN-222CJVABR
- JP1, JP2: device pinhead:PINHD-2X8 -> pinhead:PINHD-2X10
Connections:
- new net +3.3V: JP2.18, U$6.VCC
- new net N$1: U$6.P11, U$8.1, U$8.2
- new net N$2: U$6.P15, U$7.1, U$7.2
- new net SCL: JP2.2, U$6.SCL
- new net SDA: JP2.1, U$6.SDA
- net +5V: now also JP1.17, JP1.18; no longer JP1.13, JP1.14
- net GND: now also JP1.19, JP1.20, U$6.A0, U$6.A1, U$6.GND, U$7.3, U$7.4, U$8.3, U$8.4; no longer JP1.15, JP1.16
- net MUTP: now also JP1.14; no longer JP1.10
- net MUTR: now also JP1.13; no longer JP1.9
- net POE+: now also JP1.16; no longer JP1.12
- net POE-: now also JP1.15; no longer JP1.11
- net VLDN: now also JP1.11; no longer JP1.7
- net VLUP: now also JP1.12; no longer JP1.8

Commit message: Added a motor Driver
Parts:
- added 1A, 1B, 2A, 2B: TP1R, pm-labs:TP1R
- added C1, C2: 1u, pm-labs:C0603R
- added R1, R2: 10k, pm-labs:R0603R
- added R3, R4: 8k, pm-labs:R0603R
- added U$9: DRIVER_LV8716QA-MH, PiProject:DRIVER_LV8716QA-MH
Connections:
- new net N$10: 2A.1, U$9.OUT2A
- new net N$11: 2B.1, U$9.OUT2B
- new net N$12: 1B.1, U$9.OUT1B
- new net N$13: 1A.1, U$9.OUT1A
- new net N$3: R4.1, U$9.RCS2
- new net N$4: R3.1, U$9.RCS1
- new net N$5: U$6.P00, U$9.IN1
- new net N$6: U$6.P01, U$9.IN2
- new net N$7: U$6.P02, U$9.IN3
- new net N$8: U$6.P03, U$9.IN4
- new net N$9: U$6.P04, U$9.PS
- net +3.3V: now also R1.2, R2.2
- net +5V: now also C1.1, C2.2, U$9.VM1, U$9.VM2
- net GND: now also C1.2, C2.1, R3.2, R4.2, U$9.GND, U$9.GND2, U$9.PGND1, U$9.PGND2
- net N$1: now also R1.1, U$6.P14; no longer U$6.P11
- net N$2: now also R2.1
Other:
- moved on the sheet: JP2

Commit message: Missing Reset Pin on I2C Gpio Expander
GPIO expander stuck in permanent reset because RST pin needs to be connected to VCC
Parts:
- added C3: (no value), pm-labs:C0603R
Connections:
- net +3.3V: now also C3.1, U$6.!RST
- net GND: now also C3.2
Changed lines of the file:
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@@
 <part name="C1" library="pm-labs" deviceset="C" device="0603R" value="1u"/>
 <part name="C2" library="pm-labs" deviceset="C" device="0603R" value="1u"/>
+<part name="C3" library="pm-labs" deviceset="C" device="0603R"/>
 </parts>
 <sheets>
@@
 <attribute name="NAME" x="91.059" y="62.484" size="1.778" layer="95" rot="R90"/>
 <attribute name="VALUE" x="96.139" y="62.484" size="1.778" layer="96" rot="R90"/>
+</instance>
+<instance part="C3" gate="G$1" x="83.82" y="-5.08" smashed="yes" rot="R90">
+<attribute name="NAME" x="83.439" y="-3.556" size="1.778" layer="95" rot="R90"/>
+<attribute name="VALUE" x="88.519" y="-3.556" size="1.778" layer="96" rot="R90"/>
 </instance>
 </instances>
@@
 <wire x1="91.44" y1="0" x2="91.44" y2="-5.08" width="0.1524" layer="91"/>
 <pinref part="SUPPLY4" gate="GND" pin="GND"/>
+<pinref part="C3" gate="G$1" pin="2"/>
+<wire x1="88.9" y1="-5.08" x2="91.44" y2="-5.08" width="0.1524" layer="91"/>
+<junction x="91.44" y="-5.08"/>
 </segment>
 <segment>
@@
 <segment>
 <pinref part="U$6" gate="G$1" pin="VCC"/>
-<wire x1="81.28" y1="0" x2="81.28" y2="-7.62" width="0.1524" layer="91"/>
+<wire x1="81.28" y1="0" x2="81.28" y2="-5.08" width="0.1524" layer="91"/>
+<wire x1="81.28" y1="-5.08" x2="81.28" y2="-7.62" width="0.1524" layer="91"/>
 <wire x1="81.28" y1="-7.62" x2="83.82" y2="-7.62" width="0.1524" layer="91"/>
-<wire x1="83.82" y1="-7.62" x2="83.82" y2="-35.56" width="0.1524" layer="91"/>
+<wire x1="83.82" y1="-7.62" x2="83.82" y2="-15.24" width="0.1524" layer="91"/>
 <label x="81.28" y="-7.62" size="1.778" layer="95" rot="R90"/>
 <pinref part="JP2" gate="A" pin="18"/>
+<wire x1="83.82" y1="-15.24" x2="83.82" y2="-35.56" width="0.1524" layer="91"/>
 <wire x1="76.2" y1="-35.56" x2="83.82" y2="-35.56" width="0.1524" layer="91"/>
-</segment>
-<segment>
+<pinref part="C3" gate="G$1" pin="1"/>
+<junction x="81.28" y="-5.08"/>
+<pinref part="U$6" gate="G$1" pin="!RST"/>
+<wire x1="96.52" y1="0" x2="96.52" y2="-15.24" width="0.1524" layer="91"/>
+<wire x1="96.52" y1="-15.24" x2="83.82" y2="-15.24" width="0.1524" layer="91"/>
+<junction x="83.82" y="-15.24"/>
+</segment>
+<segment>
