File: DaughterBoard/DaughterBoard.brd (EAGLE design)
At the start: 27.6 x 20.9 mm, 6 parts

Commit message: Finished modified daughterboard
Parts:
- added JP2: (no value), pinhead:2X08
- JP1: device pinhead:2X04 -> pinhead:2X08
- moved U$5 34.6 mm to (-6.60, -9.50), turned to 90 degrees
- moved U$3 30.6 mm to (-6.60, -17.0), turned to 90 degrees
- moved U$4 27.1 mm to (6.70, -16.9)
- moved U$2 17.8 mm to (6.70, -9.50)
- moved U$1 15.8 mm to (-1.90, 9.40), flipped to the top, turned to 0 degrees
- moved JP1 9.62 mm to (0.00, 25.4), turned to 180 degrees
Connections:
- net +5V: now also JP1.13, JP1.14; no longer JP1.4
- net GND: now also JP1.15, JP1.16; no longer JP1.2
- net MUTP: now also JP1.10, U$5.3, U$5.4; no longer JP1.5, U$4.3, U$4.4
- net MUTR: now also JP1.9, U$3.3, U$3.4; no longer JP1.1, U$2.3, U$2.4
- net POE+: now also JP1.12; no longer JP1.8
- net POE-: now also JP1.11; no longer JP1.6
- net VLDN: now also JP1.7, U$2.3, U$2.4; no longer JP1.3, U$3.3, U$3.4
- net VLUP: now also JP1.8, U$4.3, U$4.4; no longer JP1.7, U$5.3, U$5.4
Routing:
- net MUTR: track 13.1 -> 56.0 mm
- net MUTP: track 15.8 -> 45.6 mm
- net VLDN: track 12.4 -> 42.0 mm
- net GND: track 0.00 -> 28.0 mm, vias 0 -> 3
- net VLUP: track 19.5 -> 46.2 mm
- net POE-: track 26.3 -> 40.3 mm
- net POE+: track 18.0 -> 27.7 mm
- net +5V: track 6.74 -> 6.20 mm
- added copper zone on layer 16, net GND
- removed copper zone on layer 1, net GND
Other:
- board size 27.6 x 20.9 mm -> 21.5 x 54.5 mm

Commit message: minor fix
Parts:
- moved U$3 0.50 mm to (-6.60, -16.5)
- moved U$4 0.40 mm to (6.70, -16.5)
Routing:
- net MUTR: track 56.0 -> 55.5 mm
Changed lines of the file:
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@@
 <element name="U$1" library="PicoDaughterBoard" package="MYBSP00502ABF" value="MYBSP00502ABF" x="-1.9" y="9.4" smashed="yes"/>
 <element name="U$2" library="PicoDaughterBoard" package="BTN-22CJVABR" value="BTN-222CJVABR" x="6.7" y="-9.5" smashed="yes" rot="R270"/>
-<element name="U$3" library="PicoDaughterBoard" package="BTN-22CJVABR" value="BTN-222CJVABR" x="-6.6" y="-17" smashed="yes" rot="R90"/>
-<element name="U$4" library="PicoDaughterBoard" package="BTN-22CJVABR" value="BTN-222CJVABR" x="6.7" y="-16.9" smashed="yes" rot="R270"/>
+<element name="U$3" library="PicoDaughterBoard" package="BTN-22CJVABR" value="BTN-222CJVABR" x="-6.6" y="-16.5" smashed="yes" rot="R90"/>
+<element name="U$4" library="PicoDaughterBoard" package="BTN-22CJVABR" value="BTN-222CJVABR" x="6.7" y="-16.5" smashed="yes" rot="R270"/>
 <element name="U$5" library="PicoDaughterBoard" package="BTN-22CJVABR" value="BTN-222CJVABR" x="-6.6" y="-9.5" smashed="yes" rot="R90"/>
 <element name="JP1" library="pinhead" library_urn="urn:adsk.eagle:library:325" package="2X08" package3d_urn="urn:adsk.eagle:package:22481/2" value="" x="0" y="25.4" smashed="yes" rot="R180">
@@
 <signal name="GND">
 <polygon width="0.1524" layer="16">
-<vertex x="11.3" y="29"/>
-<vertex x="-10.9" y="29"/>
-<vertex x="-10.9" y="-27.6"/>
-<vertex x="11.3" y="-27.6"/>
+<vertex x="10.8" y="28.5"/>
+<vertex x="-10.7" y="28.5"/>
+<vertex x="-10.7" y="-26"/>
+<vertex x="10.8" y="-26"/>
 </polygon>
 <contactref element="JP1" pad="15"/>
@@
 <contactref element="U$1" pad="3"/>
 <wire x1="-8.85" y1="-7" x2="-8.85" y2="-12" width="0.2" layer="1"/>
-<wire x1="-8.85" y1="-19.5" x2="-8.85" y2="-14.5" width="0.2" layer="1"/>
-<wire x1="8.95" y1="-19.4" x2="8.95" y2="-14.4" width="0.2" layer="1"/>
+<wire x1="-8.85" y1="-19" x2="-8.85" y2="-14" width="0.2" layer="1"/>
+<wire x1="8.95" y1="-19" x2="8.95" y2="-14" width="0.2" layer="1"/>
 <wire x1="8.95" y1="-7" x2="8.95" y2="-12" width="0.2" layer="1"/>
-<wire x1="8.95" y1="-12" x2="8.1" y2="-12.85" width="0.2" layer="1"/>
-<wire x1="8.1" y1="-12.85" x2="8.1" y2="-13.2" width="0.2" layer="1"/>
-<via x="8.1" y="-13.2" extent="1-16" drill="0.35"/>
-<wire x1="8.95" y1="-14.4" x2="8.1" y2="-13.55" width="0.2" layer="1"/>
-<wire x1="8.1" y1="-13.55" x2="8.1" y2="-13.2" width="0.2" layer="1"/>
-<wire x1="-8.85" y1="-14.5" x2="-7.9" y2="-13.55" width="0.2" layer="1"/>
-<wire x1="-7.9" y1="-13.55" x2="-7.9" y2="-13.3" width="0.2" layer="1"/>
-<via x="-7.9" y="-13.3" extent="1-16" drill="0.35"/>
-<wire x1="-8.85" y1="-12" x2="-7.9" y2="-12.95" width="0.2" layer="1"/>
-<wire x1="-7.9" y1="-12.95" x2="-7.9" y2="-13.3" width="0.2" layer="1"/>
-<wire x1="3.6" y1="20.9" x2="5.2" y2="20.9" width="0.2" layer="1"/>
-<via x="5.2" y="20.9" extent="1-16" drill="0.35"/>
+<wire x1="8.95" y1="-12" x2="7.95" y2="-13" width="0.2" layer="1"/>
+<wire x1="7.95" y1="-13" x2="7.8" y2="-13" width="0.2" layer="1"/>
+<via x="7.8" y="-13" extent="1-16" drill="0.35"/>
+<wire x1="8.95" y1="-14" x2="7.95" y2="-13" width="0.2" layer="1"/>
+<wire x1="-7.7" y1="-13" x2="-7.85" y2="-13" width="0.2" layer="1"/>
+<wire x1="-7.85" y1="-13" x2="-8.85" y2="-14" width="0.2" layer="1"/>
+<via x="-7.7" y="-13" extent="1-16" drill="0.35"/>
+<wire x1="-8.85" y1="-12" x2="-7.85" y2="-13" width="0.2" layer="1"/>
+<wire x1="3.6" y1="20.9" x2="5.4" y2="20.9" width="0.2" layer="1"/>
+<via x="5.4" y="20.9" extent="1-16" drill="0.35"/>
 </signal>
 <signal name="+5V">
@@
 <contactref element="JP1" pad="11"/>
 <contactref element="U$1" pad="2"/>
-<wire x1="3.6" y1="-2.1" x2="-4.8476" y2="-2.1" width="0.2" layer="1"/>
-<wire x1="-4.8476" y1="-2.1" x2="-7.0476" y2="0.1" width="0.2" layer="1"/>
-<wire x1="-7.0476" y1="0.1" x2="-7.0476" y2="18.70001875" width="0.2" layer="1"/>
-<wire x1="-7.0476" y1="18.70001875" x2="-2.7956" y2="22.95201875" width="0.2" layer="1"/>
-<wire x1="-2.7956" y1="22.95201875" x2="-2.7956" y2="24.55018125" width="0.2" layer="1"/>
-<wire x1="-3.81" y1="25.56458125" x2="-3.81" y2="26.67" width="0.2" layer="1"/>
-<wire x1="-2.7956" y1="24.55018125" x2="-3.81" y2="25.56458125" width="0.2" layer="1"/>
+<wire x1="3.6" y1="-2.1" x2="-4.8476" y2="-2.1" width="0.5" layer="1"/>
+<wire x1="-4.8476" y1="-2.1" x2="-6.7476" y2="-0.2" width="0.5" layer="1"/>
+<wire x1="-6.7476" y1="-0.2" x2="-6.7476" y2="18.20001875" width="0.5" layer="1"/>
+<wire x1="-6.7476" y1="18.20001875" x2="-2.5956" y2="22.35201875" width="0.5" layer="1"/>
+<wire x1="-2.5956" y1="22.35201875" x2="-2.5956" y2="24.65018125" width="0.5" layer="1"/>
+<wire x1="-3.81" y1="25.86458125" x2="-3.81" y2="26.67" width="0.5" layer="1"/>
+<wire x1="-2.5956" y1="24.65018125" x2="-3.81" y2="25.86458125" width="0.5" layer="1"/>
 </signal>
 <signal name="MUTR">
@@
 <contactref element="U$3" pad="4"/>
 <contactref element="U$3" pad="3"/>
-<wire x1="-4.35" y1="-19.5" x2="-4.35" y2="-14.5" width="0.2" layer="1"/>
-<wire x1="-4.35" y1="-14.5" x2="-4.35" y2="-13.75695" width="0.2" layer="1"/>
+<wire x1="-4.35" y1="-19" x2="-4.35" y2="-14" width="0.2" layer="1"/>
+<wire x1="-4.35" y1="-14" x2="-4.35" y2="-13.75695" width="0.2" layer="1"/>
 <wire x1="-4.35" y1="-13.75695" x2="-3.4476" y2="-12.85455" width="0.2" layer="1"/>
 <wire x1="-3.4476" y1="-12.85455" x2="-3.4476" y2="-6.595975" width="0.2" layer="1"/>
@@
 <wire x1="4.34758125" y1="-3.9048" x2="5.4048" y2="-2.84758125" width="0.2" layer="1"/>
 <wire x1="5.4048" y1="-2.84758125" x2="5.4048" y2="-1.35241875" width="0.2" layer="1"/>
-<wire x1="-1.27" y1="25.56458125" x2="-1.27" y2="26.67" width="0.2" layer="1"/>
-<wire x1="-0.2556" y1="24.55018125" x2="-1.27" y2="25.56458125" width="0.2" layer="1"/>
-<wire x1="-0.2556" y1="4.30798125" x2="-0.2556" y2="24.55018125" width="0.2" layer="1"/>
+<wire x1="-1.27" y1="25.66458125" x2="-1.27" y2="26.67" width="0.2" layer="1"/>
+<wire x1="-0.2" y1="24.59458125" x2="-1.27" y2="25.66458125" width="0.2" layer="1"/>
+<wire x1="-0.2" y1="4.25238125" x2="-0.2" y2="24.59458125" width="0.2" layer="1"/>
 <wire x1="-3.4476" y1="-6.595975" x2="-0.756425" y2="-3.9048" width="0.2" layer="1"/>
-<wire x1="5.4048" y1="-1.35241875" x2="-0.2556" y2="4.30798125" width="0.2" layer="1"/>
+<wire x1="5.4048" y1="-1.35241875" x2="-0.2" y2="4.25238125" width="0.2" layer="1"/>
 </signal>
 <signal name="VLDN">
@@
 <wire x1="4.45" y1="-12" x2="4.45" y2="-7" width="0.2" layer="1"/>
 <wire x1="5.7572" y1="-2.99355625" x2="5.7572" y2="-1.20644375" width="0.2" layer="1"/>
-<wire x1="5.7572" y1="-1.20644375" x2="0.0968" y2="4.45395625" width="0.2" layer="1"/>
+<wire x1="5.7572" y1="-1.20644375" x2="0.2" y2="4.35075625" width="0.2" layer="1"/>
 <wire x1="4.45" y1="-7" x2="4.45" y2="-4.30075625" width="0.2" layer="1"/>
 <wire x1="4.45" y1="-4.30075625" x2="5.7572" y2="-2.99355625" width="0.2" layer="1"/>
-<wire x1="0.0968" y1="25.4968" x2="1.27" y2="26.67" width="0.2" layer="1"/>
-<wire x1="0.0968" y1="4.45395625" x2="0.0968" y2="25.4968" width="0.2" layer="1"/>
+<wire x1="0.2" y1="25.6" x2="1.27" y2="26.67" width="0.2" layer="1"/>
+<wire x1="0.2" y1="4.35075625" x2="0.2" y2="25.6" width="0.2" layer="1"/>
 </signal>
 <signal name="VLUP">
@@
 <contactref element="U$4" pad="4"/>
 <contactref element="U$4" pad="3"/>
-<wire x1="4.45" y1="-19.4" x2="4.45" y2="-14.4" width="0.2" layer="1"/>
-<wire x1="1.27" y1="3.77913125" x2="1.27" y2="24.13" width="0.2" layer="1"/>
-<wire x1="6.1096" y1="-1.06046875" x2="1.27" y2="3.77913125" width="0.2" layer="1"/>
+<wire x1="4.45" y1="-19" x2="4.45" y2="-14" width="0.2" layer="1"/>
+<wire x1="0.6" y1="23.46" x2="0.6" y2="4.44913125" width="0.2" layer="1"/>
+<wire x1="0.6" y1="23.46" x2="1.27" y2="24.13" width="0.2" layer="1"/>
+<wire x1="6.1096" y1="-1.06046875" x2="0.6" y2="4.44913125" width="0.2" layer="1"/>
 <wire x1="6.1096" y1="-12.09735" x2="6.1096" y2="-1.06046875" width="0.2" layer="1"/>
-<wire x1="4.45" y1="-14.4" x2="4.45" y2="-13.75695" width="0.2" layer="1"/>
+<wire x1="4.45" y1="-14" x2="4.45" y2="-13.75695" width="0.2" layer="1"/>
 <wire x1="4.45" y1="-13.75695" x2="6.1096" y2="-12.09735" width="0.2" layer="1"/>
 </signal>
@@
 <wire x1="5.0524" y1="-2.70160625" x2="5.0524" y2="-1.49839375" width="0.2" layer="1"/>
 <wire x1="-4.35" y1="-7" x2="-0.9024" y2="-3.5524" width="0.2" layer="1"/>
-<wire x1="-1.27" y1="4.82400625" x2="-1.27" y2="24.13" width="0.2" layer="1"/>
+<wire x1="-0.67" y1="23.53" x2="-0.67" y2="4.22400625" width="0.2" layer="1"/>
+<wire x1="-0.67" y1="23.53" x2="-1.27" y2="24.13" width="0.2" layer="1"/>
 <wire x1="-0.9024" y1="-3.5524" x2="4.20160625" y2="-3.5524" width="0.2" layer="1"/>
-<wire x1="5.0524" y1="-1.49839375" x2="-1.27" y2="4.82400625" width="0.2" layer="1"/>
+<wire x1="5.0524" y1="-1.49839375" x2="-0.67" y2="4.22400625" width="0.2" layer="1"/>
 </signal>
 <signal name="POE+">
 <contactref element="JP1" pad="12"/>
 <contactref element="U$1" pad="1"/>
-<wire x1="-7.4" y1="-2.1" x2="-7.4" y2="18.3" width="0.2" layer="1"/>
-<wire x1="-3.81" y1="24.13" x2="-3.81" y2="22.43599375" width="0.2" layer="1"/>
-<wire x1="-3.81" y1="22.43599375" x2="-7.4" y2="18.84599375" width="0.2" layer="1"/>
-<wire x1="-7.4" y1="18.84599375" x2="-7.4" y2="18.3" width="0.2" layer="1"/>
+<wire x1="-7.4" y1="-2.1" x2="-7.4" y2="18.54599375" width="0.5" layer="1"/>
+<wire x1="-3.81" y1="24.13" x2="-3.81" y2="22.13599375" width="0.5" layer="1"/>
+<wire x1="-3.81" y1="22.13599375" x2="-7.4" y2="18.54599375" width="0.5" layer="1"/>
 </signal>
 </signals>

Commit message: Added an I2C expander
Parts:
- added U$6: GPIOEX_TCA9539PWR, PicoDaughterBoard:GPIOEX_TCA9539PWR
- added U$7, U$8: BTN-222CJVABR, PicoDaughterBoard:BTN-22CJVABR
- JP1, JP2: device pinhead:2X08 -> pinhead:2X10
- moved U$2 6.90 mm to (-0.20, -9.50), turned to 90 degrees
- moved U$4 6.90 mm to (-0.20, -16.5), turned to 90 degrees
- moved JP1 2.54 mm to (2.54, 25.4)
- moved JP2 2.54 mm to (2.54, -22.9), turned to 180 degrees
Connections:
- new net +3.3V: JP2.18, U$6.VCC
- new net N$1: U$6.P11, U$8.1, U$8.2
- new net N$2: U$6.P15, U$7.1, U$7.2
- new net SCL: JP2.2, U$6.SCL
- new net SDA: JP2.1, U$6.SDA
- net +5V: now also JP1.17, JP1.18; no longer JP1.13, JP1.14
- net GND: now also JP1.19, JP1.20, U$6.A0, U$6.A1, U$6.GND, U$7.3, U$7.4, U$8.3, U$8.4; no longer JP1.15, JP1.16
- net MUTP: now also JP1.14; no longer JP1.10
- net MUTR: now also JP1.13; no longer JP1.9
- net POE+: now also JP1.16; no longer JP1.12
- net POE-: now also JP1.15; no longer JP1.11
- net VLDN: now also JP1.11; no longer JP1.7
- net VLUP: now also JP1.12; no longer JP1.8
Routing:
- net +3.3V: track 0.00 -> 39.5 mm
- net SCL: track 0.00 -> 19.7 mm
- net GND: track 27.8 -> 44.7 mm, vias 3 -> 7
- net SDA: track 0.00 -> 16.9 mm
- net N$2: track 0.00 -> 14.4 mm
- net N$1: track 0.00 -> 7.44 mm
- net VLUP: track 46.4 -> 47.4 mm
- net VLDN: track 42.0 -> 43.0 mm
- net POE-: track 40.2 -> 39.4 mm
Other:
- board size 21.5 x 54.5 mm -> 26.5 x 54.5 mm

Commit message: Added a motor Driver
Parts:
- added 1A, 1B, 2A, 2B: TP1R, pm-labs:TP1R
- added C1, C2: 1u, pm-labs:0603R
- added R1, R2: 10k, pm-labs:0603R
- added R3, R4: 8k, pm-labs:0603R
- added U$9: DRIVER_LV8716QA-MH, PiProject:DRIVER-LV8716QA-MH
- moved U$6 2.75 mm to (10.6, 0.50)
- moved U$1 1.00 mm to (-2.90, 9.40)
Connections:
- new net N$10: 2A.1, U$9.OUT2A
- new net N$11: 2B.1, U$9.OUT2B
- new net N$12: 1B.1, U$9.OUT1B
- new net N$13: 1A.1, U$9.OU1A
- new net N$3: R4.A, U$9.RCS2
- new net N$4: R3.A, U$9.RCS1
- new net N$5: U$6.P00, U$9.IN1
- new net N$6: U$6.P01, U$9.IN2
- new net N$7: U$6.P02, U$9.IN3
- new net N$8: U$6.P03, U$9.IN4
- new net N$9: U$6.P04, U$9.PS
- net +3.3V: now also R1.B, R2.B
- net +5V: now also C1.A, C2.B, U$9.VM1, U$9.VM2
- net GND: now also C1.B, C2.A, R3.B, R4.B, U$9.GND, U$9.GND2, U$9.PGND1, U$9.PGND2
- net N$1: now also R1.A, U$6.P14; no longer U$6.P11
- net N$2: now also R2.A
Routing:
- net +5V: track 6.20 -> 47.1 mm, vias 0 -> 4
- net GND: track 44.7 -> 55.4 mm, vias 7 -> 12
- net N$10: track 0.00 -> 8.99 mm
- net N$11: track 0.00 -> 7.59 mm
- net N$12: track 0.00 -> 6.18 mm
- net N$9: track 0.00 -> 5.41 mm, vias 0 -> 2
- net POE-: track 39.4 -> 34.1 mm
- net N$13: track 0.00 -> 4.77 mm
- net N$2: track 14.4 -> 17.9 mm
- net POE+: track 27.7 -> 30.8 mm
- net N$8: track 0.00 -> 3.03 mm
- net N$1: track 7.44 -> 10.4 mm
- net +3.3V: track 39.5 -> 42.3 mm
- net N$7: track 0.00 -> 2.54 mm
- net SDA: track 16.9 -> 19.4 mm
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
Commit message: Missing Reset Pin on I2C Gpio Expander
GPIO expander stuck in permanent reset because RST pin needs to be connected to VCC
Parts:
- added C3: (no value), pm-labs:0603R
- moved R2 6.22 mm to (10.9, 0.20), turned to 270 degrees
- moved R3 5.10 mm to (13.6, 10.8)
- moved R4 5.10 mm to (8.80, 10.8)
- moved C1 5.10 mm to (8.80, 13.2)
- moved C2 5.10 mm to (13.6, 13.2)
- moved U$9 5.10 mm to (11.2, 12.1)
- moved U$6 4.91 mm to (10.9, 5.40)
- moved R1 4.62 mm to (9.70, 0.20), turned to 270 degrees
- moved 1A 3.10 mm to (14.1, 15.3)
- moved 1B 3.10 mm to (14.1, 16.5)
- moved 2B 3.10 mm to (14.1, 17.7)
- moved 2A 3.10 mm to (14.1, 18.9)
Connections:
- net +3.3V: now also C3.A, U$6.!RST
- net GND: now also C3.B
Routing:
- net +3.3V: track 42.3 -> 57.7 mm
- net +5V: track 47.1 -> 39.3 mm
- net N$1: track 10.4 -> 17.5 mm
- net N$2: track 17.9 -> 23.9 mm
- net SCL: track 22.2 -> 27.4 mm
- net SDA: track 19.4 -> 24.5 mm
- net GND: track 55.4 -> 56.4 mm, vias 12 -> 13
- net N$10: track 8.99 -> 8.06 mm
- net N$13: track 4.77 -> 3.99 mm
- net N$11: track 7.59 -> 6.95 mm

Commit message: looks better
Routing:
- net GND: track 56.4 -> 55.2 mm
- net +3.3V: track 57.7 -> 58.5 mm
Changed lines of the file:
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@@
 <contactref element="C1" pad="B"/>
 <contactref element="C2" pad="A"/>
-<wire x1="11.51305" y1="12.1" x2="11.2" y2="12.1" width="0.2" layer="1"/>
 <wire x1="10.45" y1="12.85" x2="9.84" y2="12.85" width="0.3" layer="1"/>
 <wire x1="12.56" y1="11.85" x2="11.45" y2="11.85" width="0.3" layer="1"/>
@@
 <wire x1="7.325" y1="7.325" x2="7.2" y2="7.2" width="0.2" layer="1"/>
 <via x="7.2" y="7.2" extent="1-16" drill="0.3"/>
-<wire x1="13.6" y1="10.15" x2="14.2" y2="9.55" width="0.2" layer="1"/>
-<wire x1="14.2" y1="9.55" x2="14.2" y2="9.5" width="0.2" layer="1"/>
 <via x="14.2" y="9.5" extent="1-16" drill="0.3"/>
 <wire x1="13.825" y1="8.3" x2="13.825" y2="9.125" width="0.2" layer="1"/>
@@
 <wire x1="5.9" y1="0.85" x2="7.2" y2="-0.45" width="0.4" layer="1"/>
 <wire x1="14.1" y1="1.3" x2="14.1" y2="0.75" width="0.4" layer="1"/>
-<wire x1="14.475" y1="1.675" x2="14.1" y2="1.3" width="0.4" layer="1"/>
 <wire x1="7.2205" y1="4.3" x2="5.9" y2="2.9795" width="0.4" layer="1"/>
 <wire x1="5.9" y1="2.9795" x2="5.9" y2="0.85" width="0.4" layer="1"/>
@@
 <wire x1="13.175" y1="4.3" x2="7.2205" y2="4.3" width="0.4" layer="1"/>
 <wire x1="13.175" y1="8.3" x2="13.175" y2="4.3" width="0.4" layer="1"/>
-<wire x1="14.475" y1="2.5" x2="14.475" y2="1.675" width="0" layer="19" extent="1-1"/>
+<wire x1="14.475" y1="2.5" x2="14.475" y2="1.675" width="0.4" layer="1"/>
+<wire x1="14.475" y1="1.675" x2="14.1" y2="1.3" width="0.4" layer="1"/>
 </signal>
 <signal name="N$1">
